File: Rosmo_ESC.kicad_sch (KiCad schematic)
At the start: 28 parts, among them J1 M-BUS, J2 USB_C_Receptacle_USB2.0, J3 Conn_01x06_MountingPin, J4 Conn_01x06_MountingPin, J5 Conn_01x03, J6 Conn_01x03, J7 Conn_01x02, U1 STM32G474RET6, U2 PRTR5V0U2F

Commit message: working on rosmo ESC, routing half done
Parts:
- removed J3: Conn_01x06_MountingPin, Connector_JST:JST_SH_SM06B-SRSS-TB_1x06-1MP_P1.00mm_Horizontal, symbol Connector_Generic_MountingPin:Conn_01x06_MountingPin
- removed J6: Conn_01x03, Connector_PinHeader_2.54mm:PinHeader_1x03_P2.54mm_Horizontal, symbol Connector_Generic:Conn_01x03
- removed U1: STM32G474RET6, runger:STM32G474RET6, symbol runger:STM32G474RET6
- added C1, C12, C24, C3, C4, C5, C6, C7, C8: 100nF 6.3V, Capacitor_SMD:C_0402_1005Metric, symbol Device:C_Small
- added C13: 100nF 50V 5%, Capacitor_SMD:C_0402_1005Metric, symbol Device:C_Small
- added C2: 10pF 6.3V 5%, Capacitor_SMD:C_0402_1005Metric, symbol Device:C_Small
- added C25, C26, C27, C28, C29, C30, C31, C32, C33, C34, C35, C36, C37, C38, C39, C40, C41, C42, C43, C44: 10uF 50V, Capacitor_SMD:C_0805_2012Metric, symbol Device:C_Small
- added D1: PMEG40T10ER, Diode_SMD:D_SOD-123, symbol Device:D_Small
- added D3: green, LED_SMD:LED_0402_1005Metric, symbol Device:LED_Small
- added D5: SC1333-01ETG, Diode_SMD:D_0402_1005Metric, symbol Device:D_TVS
- added D6: 2.84V, Diode_SMD:D_SOD-523, symbol Device:D_Zener_Small
- added J3: Conn_01x04_MountingPin, runger:Grove_A2006WF-04A, symbol Connector_Generic_MountingPin:Conn_01x04_MountingPin
- added J4: Conn_02x05, Connector_PinHeader_1.27mm:PinHeader_2x05_P1.27mm_Vertical_SMD, symbol Connector_Generic:Conn_02x05_Odd_Even
- added J5: JST_SH_SM06B-SRSS-TB_1x06-1MP, Connector_JST:JST_SH_SM06B-SRSS-TB_1x06-1MP_P1.00mm_Horizontal, symbol Connector_Generic_MountingPin:Conn_01x06_MountingPin
- added J8: Conn_01x03, TerminalBlock_Phoenix:TerminalBlock_Phoenix_PT-1,5-3-3.5-H_1x03_P3.50mm_Horizontal, symbol Connector_Generic:Conn_01x03
- added L1: SimpleFOC_Logo, runger:MadeForSimpleFOC_16mm, symbol runger:SimpleFOC_Logo
- added L2: Robo_Logo, runger:Robo_logo2, symbol runger:Robo_Logo
- added L3: Logo_Open_Hardware_Small, Symbol:OSHW-Symbol_6.7x6mm_SilkScreen, symbol Graphic:Logo_Open_Hardware_Small
- added L4: CC_Logo, runger:CC_Logo_5mm, symbol runger:CC_Logo
- added L5: CC_Attribution_Logo, runger:CC_Attribution_Logo_5mm, symbol runger:CC_Attribution_Logo
- added L6: CC_Sharealike_Logo, runger:CC_Sharealike_Logo_5mm, symbol runger:CC_Sharealike_Logo
- added Q1: BC847BTT1G, Package_TO_SOT_SMD:SOT-416, symbol Device:Q_NPN_BEC
- added R1, R2, R32, R33: 2k2, Resistor_SMD:R_0402_1005Metric, symbol Device:R_Small
- added R10, R11, R14, R3, R4: 5k1, Resistor_SMD:R_0402_1005Metric, symbol Device:R_Small
- added R12: 47k 1%, Resistor_SMD:R_0402_1005Metric, symbol Device:R_Small
- added R13: 10k, Resistor_SMD:R_0402_1005Metric, symbol Device:R_Small
- added R15: 300R, Resistor_SMD:R_0402_1005Metric, symbol Device:R_Small
- added R16: 2.2k 1%, Resistor_SMD:R_0402_1005Metric, symbol Device:R_Small
- added R17: 200Ω, Resistor_SMD:R_0402_1005Metric, symbol Device:R_Small
- added U1: STM32G491MET6, Package_QFP:LQFP-80_12x12mm_P0.5mm, symbol runger:STM32G491MET6
- added X1: 25MHz, Oscillator:Oscillator_SMD_Abracon_ASCO-4Pin_1.6x1.2mm, symbol Oscillator:ASCO
- J2: Port (none) -> USB-C
- J6: renamed from J4; value Conn_01x06_MountingPin -> JST_SH_SM06B-SRSS-TB_1x06-1MP; Manu (none) -> JST; Part (none) -> JST_SH_SM06B-SRSS-TB_1x06-1MP; Port (none) -> SPI Sensor 1
- J7: renamed from J5; footprint Connector_PinHeader_2.54mm:PinHeader_1x03_P2.54mm_Horizontal -> TerminalBlock_Phoenix:TerminalBlock_Phoenix_PT-1,5-3-3.5-H_1x03_P3.50mm_Horizontal; Port (none) -> Motor 0
- J9: renamed from J7; footprint Connector_PinHeader_2.54mm:PinHeader_1x02_P2.54mm_Horizontal -> TerminalBlock_Phoenix:TerminalBlock_Phoenix_PT-1,5-2-5.0-H_1x02_P5.00mm_Horizontal; Port (none) -> Power in
- renumbered C3 to C10, C1 to C11, C2 to C9, D1 to D2, D2 to D4, R1 to R5, R2 to R6, R3 to R7, R4 to R8, R5 to R9
Connections:
- net +5V: now also D4.4 (VDD), C12.2, D1.1 (K), R14.2
- net D+: now also C10.1, R5.2; no longer C9.1, R6.2
- net D-: now also C9.1, R6.2; no longer C10.1, R5.2
- net GND: now also D4.2 (VSS), J6.1 (Pin_1), J6.MP (MountPin), J9.1 (Pin_1), C1.1, C13.2, C2.1, C24.1, C25.2, C26.2, C27.2, C28.2, C29.2, C3.1, C30.2, C31.2, C32.2, C33.2, C34.2, C35.2, C36.2, C37.2, C38.2, C39.2, C4.1, C40.2, C41.2, C42.2, C43.2, C44.2, C5.1, C6.1, C7.1, C8.1, D5.1 (A1), D6.2 (A), J3.1 (Pin_1), J3.MP (MountPin), J4.3 (Pin_3), J4.5 (Pin_5), J4.9 (Pin_9), J5.1 (Pin_1), J5.MP (MountPin), R15.1, R16.1, R17.1, U1.15 (VSS), U1.27 (VSSA), U1.40 (VSS), U1.50 (VSS), U1.61 (*VSS), U1.79 (*VSS), X1.2 (GND)
- net GPIO18: now also U1.66 (*PC10)
- net GPIO19: now also U1.67 (*PC11)
- net GPIO2: now also R3.1, U1.65 (*PA15)
- net GPIO21: now also R2.1, U1.56 (PA8)
- net GPIO22: now also R1.1, U1.57 (PA9)
- net GPIO23: now also U1.68 (*PC12)
- net GPIO5: now also R4.1, U1.12 (PA0)
- net M0_AOUTU: now also U1.9 (PC1)
- net M0_ENU: now also U1.31 (PE8)
- net M0_ENV: now also U1.33 (PE10)
- net M0_ENW: now also U1.35 (PE12)
- net M0_INU: now also U1.32 (PE9)
- net M0_INV: now also U1.34 (PE11)
- net M0_INW: now also U1.36 (PE13)
- net M0_PHASEU: now also J7.1 (Pin_1)
- net M0_PHASEV: now also J7.2 (Pin_2)
- net M0_nFAULT: now also U1.39 (PB10)
- net M0_nSLEEP: now also U1.38 (PE15)
- net M1_AOUTU: now also U1.13 (PA1)
- net M1_ENU: now also U1.72 (*PB3)
- net M1_ENV: now also U1.73 (*PB4)
- net M1_ENW: now also U1.69 (*PD0)
- net M1_INU: now also U1.52 (PC6)
- net M1_INV: now also U1.53 (PC7)
- net M1_INW: now also U1.55 (PC9)
- net M1_PHASEU: now also J8.1 (Pin_1)
- net M1_PHASEV: now also J8.2 (Pin_2)
- net M1_nFAULT: now also U1.47 (PD8)
- net M1_nSLEEP: now also U1.48 (PD9)
- net VBUS: no longer D2.2 (A), FB1.2
- net VSS: now also J9.2 (Pin_2), C25.1, C26.1, C27.1, C28.1, C29.1, C30.1, C31.1, C32.1, C33.1, C34.1, C35.1, C36.1, C37.1, C38.1, C39.1, C40.1, C41.1, C42.1, C43.1, C44.1, D3.2 (A), R12.2, R13.2
- net at R6.1: now also U1.59 (PA11)
- net VDD: now reaches J6.2 (Pin_2)
- net VDD: now also C1.2, C24.2, C3.2, C4.2, C5.2, C6.2, C7.2, C8.2, J3.2 (Pin_2), J4.1 (Pin_1), J5.2 (Pin_2), R1.2, R10.2, R11.2, R2.2, R3.2, R32.2, R33.2, R4.2, U1.1 (VBAT), U1.16 (VDD), U1.29 (VDDA), U1.41 (VDD), U1.51 (VDD), U1.62 (*VDD), U1.80 (*VDD), X1.1 (Tri-State), X1.4 (VDD)
- net MOSI1: now reaches J6.3 (Pin_3)
- net MOSI1: now also U1.46 (PB15)
- net MISO1: now reaches J6.4 (Pin_4)
- net MISO1: now also U1.45 (PB14)
- net SCLK1: now reaches J6.5 (Pin_5)
- net SCLK1: now also U1.44 (PB13)
- net nCS1: now reaches J6.6 (Pin_6)
- net nCS1: now also R11.1, U1.43 (PB12)
- net at R5.1: now also U1.60 (PA12)
- net at D4.1 (DOUT): now also R15.2
- net LED: now reaches D4.3 (DIN)
- net LED: now also C12.1, R14.1, U1.42 (PB11)
- net M0_PHASEW: now reaches J7.3 (Pin_3)
- new net: D3.1 (K), Q1.3 (C)
- new net: Q1.2 (E), R17.2
- new net: D6.1 (K), Q1.1 (B), R13.1
- new net +5VD: D1.2 (A), D2.2 (A), FB1.2
- new net BOOT0: U1.77 (*PB8-BOOT0)
- new net M0_AOUTV: U1.10 (PC2)
- new net M0_AOUTW: U1.11 (PC3)
- new net M1_AOUTV: U1.14 (PA2)
- new net M1_AOUTW: U1.17 (PA3)
- new net M1_PHASEW: J8.3 (Pin_3)
- new net MISO0: J5.4 (Pin_4), U1.20 (PA6)
- new net MOSI0: J5.3 (Pin_3), U1.21 (PA7)
- new net OSCIN: C2.2, U1.5 (PF0-OSC_IN), X1.3 (OUT)
- new net SCL1: J3.4 (Pin_4), R32.1, U1.54 (PC8)
- new net SCLK0: J5.5 (Pin_5), U1.19 (PA5)
- new net SDA1: J3.3 (Pin_3), R33.1, U1.74 (*PB5)
- new net SWCLK: J4.4 (Pin_4), U1.64 (*PA14)
- new net SWDIO: J4.2 (Pin_2), U1.63 (*PA13)
- new net VBAT: C13.1, D5.2 (A2), R12.1, R16.2, U1.8 (PC0)
- new net nCS0: J5.6 (Pin_6), R10.1, U1.18 (PA4)
- new net nRST: J4.10 (Pin_10), U1.7 (PG10-NRST)
- no-connect marks 3 -> 25
Other:
- note added: "C25 to C44: 10uF 50V"
- note added: "Check if this is a good plan... We could also put a 12V buck on there to power the stack..."
- note added: "Could introduce optionality via a jumper-header, would make it easier to integrate multiple driver modules and to be compatible with other modules."
- note added: "Don’t need 32KHz clock - fast one will do. Assume 5pF stray capacitance + 10pF load capacitor = 15pF load, as required."
- note added: "Red sections denote optional functionality that could be omitted to reduce price of a production run."
- note added: "Which GPIO pins to map to? Check what other modules (e.g. CAN Bus) might be using."
- company: (none) -> Rosmo Robot
- title: (none) -> Rosmo ESC
- moved on the sheet: C10, C9, D4, J6, J7, J9, R5, R6
