File: Rosmo_ESC.kicad_sch (KiCad schematic)
At the start: 87 parts, among them J1 M-BUS, J2 USB_C_Receptacle_USB2.0, J3 Conn_01x04_MountingPin, J4 Conn_02x05, J5 JST_SH_SM06B-SRSS-TB_1x06-1MP, J6 JST_SH_SM06B-SRSS-TB_1x06-1MP, J7 Conn_01x03, J8 Conn_01x03, J9 Conn_01x02, Q1 BC847BTT1G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

Commit message: intial routing done
Connections:
- net GND: now also C12.1; no longer J3.MP (MountPin), J5.MP (MountPin), J6.MP (MountPin)
- net LED: now also U1.58 (PA10); no longer C12.1, U1.42 (PB11)
- net M0_AOUTU: now also U1.11 (PC3); no longer U1.9 (PC1)
- net M0_AOUTW: now also U1.9 (PC1); no longer U1.11 (PC3)
- net M0_nFAULT: now also U1.22 (PC4); no longer U1.39 (PB10)
- net M0_nSLEEP: now also U1.23 (PC5); no longer U1.38 (PE15)
- net VBAT: now also U1.26 (PB2); no longer U1.8 (PC0)
- no-connect marks 25 -> 28
Changed lines of the file:
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@@
   (junction (at 211.455 213.995) (diameter 0) (color 0 0 0 0))
   (junction (at 211.455 239.395) (diameter 0) (color 0 0 0 0))
-  (junction (at 212.725 142.875) (diameter 0) (color 0 0 0 0))
   (junction (at 215.265 213.995) (diameter 0) (color 0 0 0 0))
   (junction (at 215.265 239.395) (diameter 0) (color 0 0 0 0))
@@
   (junction (at 226.695 239.395) (diameter 0) (color 0 0 0 0))
   (junction (at 230.505 135.255) (diameter 0) (color 0 0 0 0))
+  (junction (at 230.505 150.495) (diameter 0) (color 0 0 0 0))
   (junction (at 230.505 213.995) (diameter 0) (color 0 0 0 0))
   (junction (at 230.505 239.395) (diameter 0) (color 0 0 0 0))
@@
   (no_connect (at 102.87 41.91))
   (no_connect (at 102.87 46.99))
-  (no_connect (at 102.87 87.63))
-  (no_connect (at 102.87 90.17))
+  (no_connect (at 102.87 52.07))
   (no_connect (at 102.87 92.71))
   (no_connect (at 102.87 95.25))
-  (no_connect (at 102.87 97.79))
   (no_connect (at 102.87 102.87))
   (no_connect (at 102.87 107.95))
   (no_connect (at 102.87 125.73))
+  (no_connect (at 102.87 128.27))
+  (no_connect (at 102.87 130.81))
   (no_connect (at 154.94 39.37))
   (no_connect (at 154.94 44.45))
@@
   (no_connect (at 154.94 57.15))
   (no_connect (at 154.94 59.69))
-  (no_connect (at 154.94 90.17))
   (no_connect (at 154.94 113.03))
+  (no_connect (at 154.94 130.81))
+  (no_connect (at 307.34 213.36))
+  (no_connect (at 318.135 184.785))
+  (no_connect (at 340.36 213.36))
   (no_connect (at 347.98 180.975))
   (no_connect (at 349.885 125.095))
@@
     (stroke (width 0) (type default) (color 0 0 0 0))
   )
-  (wire (pts (xy 196.215 142.875) (xy 212.725 142.875))
+  (wire (pts (xy 196.215 142.875) (xy 221.615 142.875))
     (stroke (width 0) (type default) (color 0 0 0 0))
   )
@@
     (stroke (width 0) (type default) (color 0 0 0 0))
   )
-  (wire (pts (xy 212.725 141.605) (xy 212.725 142.875))
+  (wire (pts (xy 212.725 141.605) (xy 212.725 150.495))
     (stroke (width 0) (type default) (color 0 0 0 0))
   )
-  (wire (pts (xy 212.725 142.875) (xy 221.615 142.875))
+  (wire (pts (xy 212.725 150.495) (xy 230.505 150.495))
     (stroke (width 0) (type default) (color 0 0 0 0))
   )
@@
     (effects (font (size 1.27 1.27)) (justify right bottom))
   )
-  (label "VBAT" (at 102.87 52.07 180)
-    (effects (font (size 1.27 1.27)) (justify right bottom))
-  )
-  (label "M0_AOUTU" (at 102.87 54.61 180)
+  (label "M0_AOUTW" (at 102.87 54.61 180)
     (effects (font (size 1.27 1.27)) (justify right bottom))
   )
@@
     (effects (font (size 1.27 1.27)) (justify right bottom))
   )
-  (label "M0_AOUTW" (at 102.87 59.69 180)
+  (label "M0_AOUTU" (at 102.87 59.69 180)
     (effects (font (size 1.27 1.27)) (justify right bottom))
   )
@@
     (effects (font (size 1.27 1.27)) (justify right bottom))
   )
+  (label "M0_nFAULT" (at 102.87 87.63 180)
+    (effects (font (size 1.27 1.27)) (justify right bottom))
+  )
+  (label "M0_nSLEEP" (at 102.87 90.17 180)
+    (effects (font (size 1.27 1.27)) (justify right bottom))
+  )
+  (label "VBAT" (at 102.87 97.79 180)
+    (effects (font (size 1.27 1.27)) (justify right bottom))
+  )
   (label "M0_ENU" (at 102.87 110.49 180)
     (effects (font (size 1.27 1.27)) (justify right bottom))
@@
     (effects (font (size 1.27 1.27)) (justify right bottom))
   )
-  (label "M0_nSLEEP" (at 102.87 128.27 180)
-    (effects (font (size 1.27 1.27)) (justify right bottom))
-  )
-  (label "M0_nFAULT" (at 102.87 130.81 180)
-    (effects (font (size 1.27 1.27)) (justify right bottom))
-  )
   (label "VBAT" (at 131.445 224.155 180)
     (effects (font (size 1.27 1.27)) (justify right bottom))
@@
     (effects (font (size 1.27 1.27)) (justify left bottom))
   )
+  (label "LED" (at 154.94 90.17 0)
+    (effects (font (size 1.27 1.27)) (justify left bottom))
+  )
   (label "SCL" (at 154.94 92.71 0)
     (effects (font (size 1.27 1.27)) (justify left bottom))
@@
     (effects (font (size 1.27 1.27)) (justify left bottom))
   )
-  (label "LED" (at 154.94 130.81 0)
-    (effects (font (size 1.27 1.27)) (justify left bottom))
-  )
   (label "BOOT0" (at 187.325 58.42 180)
     (effects (font (size 1.27 1.27)) (justify right bottom))
@@
     (pin "1")
   )
-  (symbol (lib_id "power:GND") (at 307.34 213.36 0) (unit 1)
-    (in_bom yes) (on_board yes)
-    (property "Reference" "#PWR051" (id 0) (at 307.34 219.71 0)
-      (effects (font (size 1.27 1.27)) hide)
-    )
-    (property "Value" "GND" (id 1) (at 307.34 217.17 0))
-    (property "Footprint" "" (id 2) (at 307.34 213.36 0)
-      (effects (font (size 1.27 1.27)) hide)
-    )
-    (property "Datasheet" "" (id 3) (at 307.34 213.36 0)
-      (effects (font (size 1.27 1.27)) hide)
-    )
-    (pin "1")
-  )
   (symbol (lib_id "power:GND") (at 313.055 172.085 270) (mirror x) (unit 1)
     (in_bom yes) (on_board yes)
@@
     (pin "1")
   )
-  (symbol (lib_id "power:GND") (at 318.135 184.785 0) (unit 1)
-    (in_bom yes) (on_board yes)
-    (property "Reference" "#PWR042" (id 0) (at 318.135 191.135 0)
-      (effects (font (size 1.27 1.27)) hide)
-    )
-    (property "Value" "GND" (id 1) (at 318.135 188.595 0))
-    (property "Footprint" "" (id 2) (at 318.135 184.785 0)
-      (effects (font (size 1.27 1.27)) hide)
-    )
-    (property "Datasheet" "" (id 3) (at 318.135 184.785 0)
-      (effects (font (size 1.27 1.27)) hide)
-    )
-    (pin "1")
-  )
   (symbol (lib_id "power:GND") (at 318.77 243.84 270) (mirror x) (unit 1)
     (in_bom yes) (on_board yes)
@@
     (pin "1")
   )
-  (symbol (lib_id "power:GND") (at 340.36 213.36 0) (unit 1)
-    (in_bom yes) (on_board yes)
-    (property "Reference" "#PWR052" (id 0) (at 340.36 219.71 0)
-      (effects (font (size 1.27 1.27)) hide)
-    )
-    (property "Value" "GND" (id 1) (at 340.36 217.17 0))
-    (property "Footprint" "" (id 2) (at 340.36 213.36 0)
-      (effects (font (size 1.27 1.27)) hide)
-    )
-    (property "Datasheet" "" (id 3) (at 340.36 213.36 0)
-      (effects (font (size 1.27 1.27)) hide)
-    )
-    (pin "1")
-  )
   (symbol (lib_id "power:GND") (at 344.17 50.165 0) (unit 1)
     (in_bom yes) (on_board yes)
@@
       (effects (font (size 1.27 1.27)) (justify left))
     )
-    (pin "ENC" input (at 48.895 205.74 180)
+    (pin "ENC" input (at 48.895 208.28 180)
       (effects (font (size 1.27 1.27)) (justify left))
     )
-    (pin "ENB" input (at 48.895 208.28 180)
+    (pin "ENB" input (at 48.895 205.74 180)
       (effects (font (size 1.27 1.27)) (justify left))
     )
@@
       (effects (font (size 1.27 1.27)) (justify left))
     )
-    (pin "ENC" input (at 48.895 255.27 180)
+    (pin "ENC" input (at 48.895 257.81 180)
       (effects (font (size 1.27 1.27)) (justify left))
     )
-    (pin "ENB" input (at 48.895 257.81 180)
+    (pin "ENB" input (at 48.895 255.27 180)
       (effects (font (size 1.27 1.27)) (justify left))
     )
@@
       (reference "#PWR041") (unit 1) (value "GND") (footprint "")
     )
-    (path "/ae402f92-fcec-446c-beef-c1e0b8f21ea9"
-      (reference "#PWR042") (unit 1) (value "GND") (footprint "")
-    )
     (path "/9895d7c8-61f7-499e-874c-a54cf3e88f76"
       (reference "#PWR043") (unit 1) (value "VDD") (footprint "")
@@
       (reference "#PWR050") (unit 1) (value "VSS") (footprint "")
     )
-    (path "/c3ba23b9-f62d-43e4-bcb4-b81c5c05a373"
-      (reference "#PWR051") (unit 1) (value "GND") (footprint "")
-    )
-    (path "/eb699428-0240-4898-8700-95424ae186e9"
-      (reference "#PWR052") (unit 1) (value "GND") (footprint "")
-    )
     (path "/7cf29c03-e9a0-460c-aed1-bc1b7c421927"

Commit message: updated to KiCad 6
Parts:
- removed L4: CC_Logo, runger:CC_Logo_5mm, symbol runger:CC_Logo
- removed L5: CC_Attribution_Logo, runger:CC_Attribution_Logo_5mm, symbol runger:CC_Attribution_Logo
- removed L6: CC_Sharealike_Logo, runger:CC_Sharealike_Logo_5mm, symbol runger:CC_Sharealike_Logo
- J2: Manu (none) -> HRO; Part (none) -> HRO_TYPE-C-31-M-12
- J3: Manu (none) -> Seeedstudio; Part (none) -> GR008WR-S-4P
- J4: Manu (none) -> Amphenol FCI; Part (none) -> 20021121-00010C8LF
- J7, J8: Manu (none) -> Amphenol Anytek; Part (none) -> 20020110-C034A01LF
- J9: footprint TerminalBlock_Phoenix:TerminalBlock_Phoenix_PT-1,5-2-5.0-H_1x02_P5.00mm_Horizontal -> TerminalBlock_Phoenix:TerminalBlock_Phoenix_PT-1,5-2-3.5-H_1x02_P3.50mm_Horizontal; Manu (none) -> Amphenol Anytek; Part (none) -> 20020110-C021A01LF
- U1: Manu (none) -> ST Microsystems; Notes (none) -> No need to order, I will send; Part (none) -> STM32G491MET6
Other:
- note removed: "Check if this is a good plan... We could also put a 12V buck on there to power the stack..."
- moved on the sheet: C12, C13, D3, D4, D5, D6, Q1, R12, R13, R14, R15, R16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

Commit message: v1 prototype for production
Parts:
- added C45, C46: 2.2uF 16V, Capacitor_SMD:C_0603_1608Metric, symbol Device:C_Small
- added J10: Conn_02x05, Connector_PinHeader_1.27mm:PinHeader_2x05_P1.27mm_Vertical_SMD, symbol Connector_Generic:Conn_02x05_Odd_Even
- added JB1: M-BUS, Connector_PinHeader_2.54mm:PinHeader_2x15_P2.54mm_Vertical_SMD, symbol Connector_Generic:Conn_02x15_Odd_Even
- added R34: 5k1, Resistor_SMD:R_0402_1005Metric, symbol Device:R_Small
- added U5: MIC5524-3.3YMT-T5, runger:TDFN-4-1EP_1x1mm_P0.65mm_EP0.5x0.5mm, symbol runger:MIC5524-3.3YMT-T5
- D4: Manu (none) -> Normand?; Part (none) -> SK6805-2427
- J1: Manu (none) -> Amphenol; Part (none) -> 89898-315BLF
- R12: Manu (none) -> Vishay / Dale; Part (none) -> CRCW040247K0FKEDC
- R16: Manu (none) -> Yageo; Part (none) -> RT0402DRE072K2L
Connections:
- net +3V3: now also JB1.11 (Pin_11)
- net +5V: now also C45.2, JB1.27 (Pin_27), U5.3 (EN), U5.4 (VIN)
- net +BATT: now also JB1.29 (Pin_29)
- net BOOT0: now also J10.9 (Pin_9), R34.2
- net EN: now also JB1.5 (Pin_5)
- net GND: now also C45.1, C46.1, JB1.2 (Pin_2), JB1.4 (Pin_4), JB1.6 (Pin_6), R34.1, U5.2 (GND), U5.5 (GND)
- net GPIO0: now also JB1.23 (Pin_23)
- net GPIO1: now also JB1.13 (Pin_13)
- net GPIO12: now also JB1.22 (Pin_22)
- net GPIO13: now also JB1.21 (Pin_21)
- net GPIO15: now also JB1.24 (Pin_24)
- net GPIO16: now also JB1.16 (Pin_16)
- net GPIO17: now also JB1.15 (Pin_15)
- net GPIO18: now also JB1.12 (Pin_12)
- net GPIO19: now also JB1.10 (Pin_10)
- net GPIO2: now also J10.3 (Pin_3), JB1.20 (Pin_20); no longer R3.1, U1.65 (*PA15)
- net GPIO21: now also JB1.18 (Pin_18)
- net GPIO22: now also JB1.17 (Pin_17)
- net GPIO23: now also JB1.8 (Pin_8)
- net GPIO25: now also JB1.7 (Pin_7)
- net GPIO26: now also JB1.9 (Pin_9)
- net GPIO3: now also JB1.14 (Pin_14)
- net GPIO34: now also JB1.25 (Pin_25)
- net GPIO35: now also JB1.1 (Pin_1)
- net GPIO36: now also JB1.3 (Pin_3)
- net GPIO5: now also J10.2 (Pin_2), JB1.19 (Pin_19); no longer R4.1, U1.12 (PA0)
- net VBUS: now also JB1.26 (Pin_26), JB1.28 (Pin_28), JB1.30 (Pin_30)
- net VDD: now also C46.2, J10.10 (Pin_10), J10.6 (Pin_6), J10.8 (Pin_8), U5.1 (VOUT)
- net ADDR2: now reaches U1.70 (*PD1)
- net ADDR2: now also J10.7 (Pin_7)
- net ADDR1: now reaches U1.71 (*PD2)
- net ADDR1: now also J10.5 (Pin_5)
- new net WAKE: J10.1 (Pin_1), R4.1, U1.12 (PA0)
- new net nCS2: J10.4 (Pin_4), R3.1, U1.65 (*PA15)
- no-connect marks 28 -> 26
Other:
- note added: "Duplicate header since SMD headers are 2 seperate components for front and back."
- note added: "Note: use the internal pull-downs on ADDR1 and ADDR2"
- note removed: "Could introduce optionality via a jumper-header, would make it easier to integrate multiple driver modules and to be compatible with other modules."
- moved on the sheet: C12, D1, D4, J1, R1, R14, R15, R2, R3, R4

Commit message: updated pinout diagramme
Other:
- note added: "LED pin type FT_da is 5V tolerant. Set to open drain."
Changed lines of the file:
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@@
     (effects (font (size 2 2)) (justify left bottom))
+  )
+  (text "LED pin type FT_da is 5V tolerant.\nSet to open drain."
+    (at 168.91 71.12 0)
+    (effects (font (size 1.27 1.27)) (justify left bottom))
   )
   (text "Note: use the internal\npull-downs on ADDR1 and ADDR2"
